File: HARDWARE/VHM-rev1/VHM-rev1.kicad_pcb (KiCad board)
At the start: 2 copper layers, 22 x 130 mm, 10 parts, among them J1 RJ45, J2 USB_C_Receptacle, Q1 DMG2301L, U1 TLP127, U2 CH340G, U3 ESP32-WROOM-32

Commit message: Added 3d objects and libraries
Parts:
- removed D1: B340, Diodes_SMD:D_SMC
- added D2: SB160, Diodes_SMD:D_SMA, F.Cu at (142.9, 131.2)
- added U4: TP4056, lib:TP4056_SOP-8-PP, F.Cu at (144.0, 92.8)
- added U5: FS8205A, Housings_SSOP:TSSOP-8_4.4x3mm_Pitch0.65mm, F.Cu at (154.5, 91.8)
- added U6: DW01, TO_SOT_Packages_SMD:SOT-23-6_Handsoldering, F.Cu at (156.3, 84.5)
- moved U2 6.89 mm to (144.3, 80.3)
